File: src/pcb_card.kicad_sch (KiCad schematic)
At the start: 0 parts

Commit message: feat: prototype schematic
Parts:
- added BT1: CR2032, easyeda2kicad:BAT-TH_CR2032-BS-6-1, symbol Device:Battery_Cell
- added C1, C3, C4: 0.1uF, Capacitor_SMD:C_0603_1608Metric, symbol Device:C
- added C2, C5: 4.7uF, Capacitor_SMD:C_0603_1608Metric, symbol Device:C
- added J1: UART, Connector_JST:JST_PH_B2B-PH-K_1x02_P2.00mm_Vertical, symbol Connector:Conn_01x02_Socket
- added J2: SOICbite, easyeda2kicad:SOIC_clipProgSmall, symbol Connector:Conn_01x08_Socket
- added JP1: SolderJumper_2_Open, Jumper:SolderJumper-2_P1.3mm_Open_TrianglePad1.0x1.5mm, symbol Jumper:SolderJumper_2_Open
- added R1, R4, R5: 0, Resistor_SMD:R_0805_2012Metric_Pad1.20x1.40mm_HandSolder, symbol Device:R
- added R2, R3, R6, R7: 10k, Resistor_SMD:R_0603_1608Metric, symbol Device:R
- added SW1, SW2: TS-1187A-B-A-B, easyeda2kicad:SW-SMD_4P-L5.1-W5.1-P3.70-LS6.5-TL_H1.5, symbol easyeda2kicad:TS-1187A-B-A-B
- added U1: CH32V003FxUx, Package_DFN_QFN:QFN-20-1EP_3x3mm_P0.4mm_EP1.65x1.65mm, symbol MCU_WCH_RiscV:CH32V003FxUx
- added U2: LIS3DH, Package_LGA:LGA-16_3x3mm_P0.5mm_LayoutBorder3x5y, symbol Sensor_Motion:LIS3DH
- added U3: CH32X035F8U6_C42442062, easyeda2kicad:WQFN-20_L3.0-W3.0-P0.40-TL-EP1.7, symbol easyeda2kicad:CH32X035F8U6_C42442062
Connections:
- new net: R1.2, U2.11 (INT1)
- new net +3V3: C1.1, C2.1, C3.1, C4.1, C5.1, J2.1 (Pin_1), JP1.2 (B), R2.1, R3.1, U1.6 (VDD), U2.1 (VDD_IO), U2.14 (VDD), U2.7 (SDO), U2.8 (CS), U3.1 (VDD)
- new net +BATT: BT1.1 (+), JP1.1 (A), SW1.3 (C), SW2.3 (C), U2.16 (ADC1)
- new net BTN1: R6.1, SW1.1 (A), U1.3 (PA2), U3.13 (PB11/T1C3/T2C1N_/RX1)
- new net CH_1: U1.10 (PC3), U3.2 (PA0/T2C1/CTS2/A0)
- new net CH_10: U1.18 (PD4), U3.20 (PC15/CC2/T2C3_/T1ET_)
- new net CH_11: U1.2 (PA1), U3.19 (PC14/CC1/T1C3_/T2C2_)
- new net CH_2: U1.11 (PC4), U3.3 (PA1/RTS2/T2C2/O1N2/O2N2/A1)
- new net CH_3: U1.12 (PC5), U3.4 (PA2/TX2/T2C3/O2O1/T2ET_/A2)
- new net CH_4: U1.13 (PC6), U3.5 (PA3/T2C4/O1O0/T3C1_/RX2/A3)
- new net CH_5: U1.14 (PC7), U3.6 (PA4/CS/O2O0/T3C2_/A4)
- new net CH_6: U1.5 (PD0), U3.7 (PA5/SCK/TX4_/O2N0/A5)
- new net CH_7: J2.6 (Pin_6), U1.15 (PD1), U3.8 (PA6/MISO/T3C1/T1BK_/O1N0/A6)
- new net CH_8: U1.16 (PD2), U3.9 (PA7/MOSI/T3C2/T1C1N_/O2P0/A7)
- new net CH_9: U1.17 (PD3), U3.10 (PB0/TX4/T1C2N_/O1P0/A8)
- new net EN: J2.8 (Pin_8), R1.1, R7.1, SW2.1 (A), U1.7 (PC0), U3.12 (PB3/TX3/T2C3_/T2C3N_/O2P1)
- new net GND: BT1.2 (-), C1.2, C2.2, C3.2, C4.2, C5.2, J2.4 (Pin_4), R6.2, R7.2, U1.21 (VSS), U1.4 (VSS), U2.10 (GND), U2.12 (GND), U2.5 (GND), U3.21 (GND)
- new net NRST: U1.1 (PD7)
- new net RX: R5.2, U1.20 (PD6)
- new net RX_EXT: J1.1 (Pin_1), J2.2 (Pin_2), R5.1
- new net SCL: R3.2, U1.9 (PC2), U2.4 (SPC), U3.17 (PC16/UDM/T1C4/TX4_/I2C_/RX4_/PC11)
- new net SDA: R2.2, U1.8 (PC1), U2.6 (SDI), U3.18 (PC17/UDP/TX4_/I2C_/RX4_/T1ET/PC10)
- new net SWCLK: J2.7 (Pin_7), U3.16 (PC19/DCK/T2C1_/T3C1_/I2C_/RX3_)
- new net SWDIO: J2.5 (Pin_5), U3.14 (PC18/DIO/TX3_/T2C1N_/T3C2_/I2C_)
- new net TX: R4.2, U1.19 (PD5)
- new net TX_EXT: J1.2 (Pin_2), J2.3 (Pin_3), R4.1
- no-connect marks 0 -> 6
Other:
- added sheet Led Matrix (led_matrix.kicad_sch)
- note added: "CH32V003F4U6"
- note added: "Check datasheet for remap"
- note added: "For prototyping! Only place 1 MCU!"
- note added: "I2C LSB"
- note added: "Subject to change based on routing"
- note added: "todo: swap to higher res"

Commit message: feat: prototype PCB done
Parts:
- added TP1: SCL, symbol Connector:TestPoint
- added TP2: SDA, symbol Connector:TestPoint
- U3: footprint easyeda2kicad:WQFN-20_L3.0-W3.0-P0.40-TL-EP1.7 -> Package_DFN_QFN:QFN-20-1EP_3x3mm_P0.4mm_EP1.65x1.65mm
Connections:
- net BTN1: now also U1.5 (PD0); no longer U1.3 (PA2)
- net CH_1: now also U1.3 (PA2), U3.20 (PC15/CC2/T2C3_/T1ET_); no longer U1.10 (PC3), U3.2 (PA0/T2C1/CTS2/A0)
- net CH_10: now also U1.11 (PC4), U3.7 (PA5/SCK/TX4_/O2N0/A5); no longer U1.18 (PD4), U3.20 (PC15/CC2/T2C3_/T1ET_)
- net CH_11: now also U1.10 (PC3), U3.6 (PA4/CS/O2O0/T3C2_/A4); no longer U1.2 (PA1), U3.19 (PC14/CC1/T1C3_/T2C2_)
- net CH_2: now also U1.2 (PA1), U3.19 (PC14/CC1/T1C3_/T2C2_); no longer U1.11 (PC4), U3.3 (PA1/RTS2/T2C2/O1N2/O2N2/A1)
- net CH_3: now also U1.18 (PD4), U3.2 (PA0/T2C1/CTS2/A0); no longer U1.12 (PC5), U3.4 (PA2/TX2/T2C3/O2O1/T2ET_/A2)
- net CH_4: now also U1.17 (PD3), U3.3 (PA1/RTS2/T2C2/O1N2/O2N2/A1); no longer U1.13 (PC6), U3.5 (PA3/T2C4/O1O0/T3C1_/RX2/A3)
- net CH_5: now also U1.16 (PD2), U3.4 (PA2/TX2/T2C3/O2O1/T2ET_/A2); no longer U1.14 (PC7), U3.6 (PA4/CS/O2O0/T3C2_/A4)
- net CH_6: now also J2.6 (Pin_6), U1.15 (PD1), U3.5 (PA3/T2C4/O1O0/T3C1_/RX2/A3); no longer U1.5 (PD0), U3.7 (PA5/SCK/TX4_/O2N0/A5)
- net CH_7: now also U1.14 (PC7), U3.10 (PB0/TX4/T1C2N_/O1P0/A8); no longer J2.6 (Pin_6), U1.15 (PD1), U3.8 (PA6/MISO/T3C1/T1BK_/O1N0/A6)
- net CH_8: now also U1.13 (PC6); no longer U1.16 (PD2)
- net CH_9: now also U1.12 (PC5), U3.8 (PA6/MISO/T3C1/T1BK_/O1N0/A6); no longer U1.17 (PD3), U3.10 (PB0/TX4/T1C2N_/O1P0/A8)
- net EN: no longer J2.8 (Pin_8)
- net NRST: now also J2.8 (Pin_8)
- net RX: now also U3.11 (PB1/T1C3N_/RX4/O2N1/A9)
- net SCL: now also TP1.1
- net SDA: now also TP2.1

Commit message: chore: breaks out I2C pins
Parts:
- TP1, TP2: footprint (none) -> TestPoint:TestPoint_Pad_D2.0mm; now fitted
Changed lines of the file:
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@@
 		(exclude_from_sim no)
 		(in_bom no)
-		(on_board no)
-		(in_pos_files yes)
-		(dnp yes)
+		(on_board yes)
+		(in_pos_files yes)
+		(dnp no)
 		(fields_autoplaced yes)
 		(property "Reference" "TP2"
@@
 			)
 		)
-		(property "Footprint" ""
+		(property "Footprint" "TestPoint:TestPoint_Pad_D2.0mm"
 			(at 153.67 161.29 0)
 			(hide yes)
@@
 		(exclude_from_sim no)
 		(in_bom no)
-		(on_board no)
-		(in_pos_files yes)
-		(dnp yes)
+		(on_board yes)
+		(in_pos_files yes)
+		(dnp no)
 		(fields_autoplaced yes)
 		(property "Reference" "TP1"
@@
 			)
 		)
-		(property "Footprint" ""
+		(property "Footprint" "TestPoint:TestPoint_Pad_D2.0mm"
 			(at 144.78 161.29 0)
 			(hide yes)
